File: hardware/smart_port.kicad_sch (KiCad schematic)
At the start: 9 parts, among them J4 4P4C, U4 SN65HVD1782DR

Commit message: relayout board
Parts:
- removed D3, D4: D_TVS, symbol Device:D_TVS
- added D13: CESD3V3AP, Package_TO_SOT_SMD:SOT-23, symbol Device:D_TVS_Dual_AAC
- R1, R2: footprint (none) -> Resistor_SMD:R_0603_1608Metric
Connections:
- net A: now also D13.1 (A1)
- net B: now also D13.2 (A2)
- net GND: now also D13.3 (common)
Other:
- moved on the sheet: R1, R2
