File: hardware/usb_port.kicad_sch (KiCad schematic)
At the start: 18 parts, among them J5 USB_C_Receptacle_USB2.0_16P, Q1 MMBT3904, Q2 MMBT3904, SW1 SW_Push, SW2 SW_Push, U6 CH340K

Commit message: relayout board
Parts:
- removed R14, R16: 1k, Resistor_SMD:R_0603_1608Metric, symbol Device:R
- renumbered R15 to R14
Connections:
- net BOOT: now also SW1.2
- net EN: now also SW2.2
Other:
- moved on the sheet: R13, R14
